File: Hardware/LilyPad_USB_Plus_Standalone.sch (EAGLE design)
At the start: 74 parts, among them J1 SEWTAP_LONG-2SIDE, J10 SEWTAP_LONG-2SIDE, J11 SEWTAP_LONG-2SIDE, J12 SEWTAP_LONG-2SIDE, J13 SEWTAP_LONG-2SIDE, J14 SEWTAP_LONG-2SIDE, J15 AMP FCI 10103594-0001LF, J2 SEWTAP_LONG-2SIDE, J3 SEWTAP_LONG-2SIDE, J4 SEWTAP_LONG-2SIDE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

Commit message: Updated schematic
Added a note for the user to clarify net naming convention and a GPIO table to the documentation folder for even further clarification.
Other:
- note added: "Note: All GPIO have digital functionality and are labled with a "D" convention. Check the product's documentation folder in this repository for more information on GPIO."
Changed lines of the file:
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@@
 3.3-4.2V on battery connector.</text>
 <text x="148.844" y="7.112" size="2.54" layer="94">Revised by: Elias Santistevan</text>
+<wire x1="76.2" y1="182.88" x2="76.2" y2="167.64" width="0.2032" layer="97" style="shortdash"/>
+<wire x1="76.2" y1="167.64" x2="88.9" y2="167.64" width="0.2032" layer="97" style="shortdash"/>
+<wire x1="88.9" y1="167.64" x2="144.78" y2="167.64" width="0.2032" layer="97" style="shortdash"/>
+<wire x1="144.78" y1="167.64" x2="144.78" y2="182.88" width="0.2032" layer="97" style="shortdash"/>
+<wire x1="144.78" y1="182.88" x2="76.2" y2="182.88" width="0.2032" layer="97" style="shortdash"/>
+<text x="78.74" y="170.18" size="1.778" layer="97">Note: All GPIO have digital functionality and
+are labled with a "D" convention. Check the
+product's documentation folder in this
+repository for more information on GPIO.</text>
+<wire x1="88.9" y1="162.56" x2="88.9" y2="167.64" width="0.2032" layer="97" style="shortdash"/>
 </plain>
 <instances>

Commit message: Post designe review changes
Other:
- note added: "Note: All GPIO have digital functionality and are labled with a "D" convention. Check the product's documentation folder in this repository for more information on GPIO. This information is also in our hookup guide."
- note added: "v10"
- note removed: "Note: All GPIO have digital functionality and are labled with a "D" convention. Check the product's documentation folder in this repository for more information on GPIO."
- note removed: "v01"
Changed lines of the file:
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@@
 <text x="220.98" y="151.13" size="1.27" layer="97">MIC5219 BYPASS</text>
 <text x="171.45" y="11.43" size="2.54" layer="94">Marshall Taylor</text>
-<text x="238.252" y="7.112" size="2.54" layer="94">v01</text>
+<text x="238.252" y="7.112" size="2.54" layer="94">v10</text>
 <text x="149.86" y="38.1" size="2.54" layer="94">LilyPad concept and shapes by:
 L. Buechley and N. Seidle</text>
@@
 3.3-4.2V on battery connector.</text>
 <text x="148.844" y="7.112" size="2.54" layer="94">Revised by: Elias Santistevan</text>
-<wire x1="76.2" y1="182.88" x2="76.2" y2="167.64" width="0.2032" layer="97" style="shortdash"/>
-<wire x1="76.2" y1="167.64" x2="88.9" y2="167.64" width="0.2032" layer="97" style="shortdash"/>
-<wire x1="88.9" y1="167.64" x2="144.78" y2="167.64" width="0.2032" layer="97" style="shortdash"/>
-<wire x1="144.78" y1="167.64" x2="144.78" y2="182.88" width="0.2032" layer="97" style="shortdash"/>
-<wire x1="144.78" y1="182.88" x2="76.2" y2="182.88" width="0.2032" layer="97" style="shortdash"/>
-<text x="78.74" y="170.18" size="1.778" layer="97">Note: All GPIO have digital functionality and
+<wire x1="76.2" y1="182.88" x2="76.2" y2="165.1" width="0.2032" layer="97" style="shortdash"/>
+<wire x1="76.2" y1="165.1" x2="88.9" y2="165.1" width="0.2032" layer="97" style="shortdash"/>
+<wire x1="88.9" y1="165.1" x2="147.32" y2="165.1" width="0.2032" layer="97" style="shortdash"/>
+<wire x1="147.32" y1="165.1" x2="147.32" y2="182.88" width="0.2032" layer="97" style="shortdash"/>
+<wire x1="147.32" y1="182.88" x2="76.2" y2="182.88" width="0.2032" layer="97" style="shortdash"/>
+<text x="78.74" y="167.64" size="1.778" layer="97">Note: All GPIO have digital functionality and
 are labled with a "D" convention. Check the
 product's documentation folder in this
-repository for more information on GPIO.</text>
-<wire x1="88.9" y1="162.56" x2="88.9" y2="167.64" width="0.2032" layer="97" style="shortdash"/>
+repository for more information on GPIO.
+This information is also in our hookup guide.</text>
+<wire x1="88.9" y1="162.56" x2="88.9" y2="165.1" width="0.2032" layer="97" style="shortdash"/>
 </plain>
 <instances>

Commit message: Changes after double check
Other:
- note added: "LilyPad USB Plus Standalone"
- note added: "Petal 2"
- note added: "Petal 3"
- note added: "Petal 4"
- note removed: "LilyPad Prototyping Board"
- note removed: "Microcontroller"
- note removed: "Petal 2 -- LUX"
- note removed: "Petal 3 -- BZR"
- note removed: "Petal 4 -- BTN"
- moved on the sheet: D10, LED2, LED3, LED4, LED5, LED6, LED7, LED8, LED9, R10, R11, R12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
